File: kicad/kicad.sch (KiCad schematic (older format))
At the start: 17 parts, among them IC1 IQRF_(DC)TR-72D, J1 Screw_Terminal_1x02, J2 Screw_Terminal_1x02, Q1 BSS138, Q2 BSS138, SW1 BondSW, U1 MeanWell_IRM-02

Commit message: Add PCB
Signed-off-by: Roman3349 <ondracek.roman@centrum.cz>
Parts:
- added C1: 100n, Capacitors_SMD:C_1206_HandSoldering, symbol C
- J1, J2: footprint Terminal_Blocks:TerminalBlock_Pheonix_MKDS1.5-2pol -> Connectors_Terminal_Blocks:TerminalBlock_DG300-7.5-02P_RM7.5mm_2pol
- RV1, RV2: footprint Varistors:RV_Disc_D7_W3.5_P5 -> Varistors:RV_Disc_D12_W3.9_P7.5
- renumbered D2 to D3
Connections:
- net +5V: now also C1.2
- net GND: now also C1.1
- net Lin: now also RL2.3, RV2.1; no longer RL2.2, RV2.2
- net Lout: now also RL2.2, RV2.2; no longer RL2.3, RV2.1
- net Lswitch: now also IC1.2 (IO/Vout); no longer IC1.8 (IO/RX/SDO)
- net Nswitch: now also IC1.8 (IO/RX/SDO); no longer IC1.2 (IO/Vout)
- net Lcurrent: now reaches IC1.1 (IO/ADC/Cin)
- no-connect marks 3 -> 2
Other:
- moved on the sheet: D1, D3, F1, IC1, J1, J2, Q1, Q2, R1, R2, RL1, RL2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

Commit message: Update schematic
Signed-off-by: Roman3349 <ondracek.roman@centrum.cz>
Parts:
- removed IC1: IQRF_(DC)TR-72D, Connectors:IQRF_KON-SIM-01, symbol IQRF_(DC)TR-72D
- removed U1: MeanWell_IRM-02, Converters_DCDC_ACDC:ACDC-Converter_MeanWell-IRM-02-x, symbol MeanWell_IRM-02
- added IC1: DCTR-72D, Connectors:IQRF_KON-SIM-01, symbol DCTR-72D
- added U1: IRM-02, Converters_DCDC_ACDC:ACDC-Converter_MeanWell-IRM-02-x, symbol IRM-02
- renumbered D3 to D2
Connections:
- net +5V: now also IC1.3 (Vin), U1.4 (+Vout)
- net GND: now also IC1.4 (GND), IC1.9 (GND), U1.3 (-Vout)
- net Lin: now also U1.2 (AC/L)
- net Lswitch: now also IC1.2 (RC2/Vout)
- net Nin: now also U1.1 (AC/N)
- net Nswitch: now also IC1.8 (RC5/RC7/RX/SDO)
- net at SW1.1: now also IC1.5 (RA5/RB4/RC6/AN4/AN11/TX/~SS~/C2OUT/CCP3)
- no-connect marks 2 -> 3
Other:
- moved on the sheet: C1, D1, D2, F1, J1, J2, Q1, Q2, R1, R2, RL1, RL2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

Commit message: Update schematic of Smart socket
Signed-off-by: Roman Ondráček <ondracek.roman@centrum.cz>
Parts:
- removed SW1: BondSW, Buttons_Switches_THT:SW_PUSH_6mm, symbol SW_Push
- removed U1: IRM-02, Converters_DCDC_ACDC:ACDC-Converter_MeanWell-IRM-02-x, symbol IRM-02
- added C2: 100n, Capacitors_SMD:C_1206_HandSoldering, symbol C
- added C3: 10u, Capacitors_SMD:C_1206_HandSoldering, symbol C
- added J3: CONN_01X04, Pin_Headers:Pin_Header_Straight_1x04_Pitch2.54mm, symbol CONN_01X04
- added R3: 68R, Resistors_SMD:R_1206_HandSoldering, symbol R
- added R4: 10k, Resistors_SMD:R_1206_HandSoldering, symbol R
- added U1: IRM-02-5, Converters_DCDC_ACDC:ACDC-Converter_MeanWell-IRM-02-x, symbol IRM-02-5
- added U2: LD1117S33TR, TO_SOT_Packages_SMD:SOT-223, symbol LD1117S33TR
- D1, D2: footprint Diodes_THT:Diode_DO-41_SOD81_Horizontal_RM10 -> Diodes_THT:D_DO-41_SOD81_P10.16mm_Horizontal
- J1, J2: footprint Connectors_Terminal_Blocks:TerminalBlock_DG300-7.5-02P_RM7.5mm_2pol -> Connectors_Terminal_Blocks:TerminalBlock_Pheonix_MKDS1.5-2pol
- LOGO1: footprint Symbols:OSHW-Logo2_9.8x8mm_Copper -> Symbols:OSHW-Logo2_7.3x6mm_SilkScreen
- RL1, RL2: footprint Relays_THT:Relay_SPST-NO_OMRON-G5Q -> Relays_THT:Relay_SPST_OMRON-G5Q
Connections:
- net labels added: +3V3, BondBtn, RelaySw
- net labels removed: Lswitch, Nswitch
- wire segments 47 -> 57
- no-connect marks 3 -> 4
Other:
- note added: "Button"
- moved on the sheet: D1, D2, F1, IC1, J1, J2, Q1, Q2, R1, R2, RL1, RL2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
